Commit message: add imu and lidar sensor

File: foxy_description/sensors/imu_generic.xacro (robot description, xacro)
@@ -1,5 +1,5 @@
 <?xml version="1.0"?>
 <robot xmlns:xacro="http://www.ros.org/wiki/xacro">
-  <xacro:macro name="rgb_camera_generic" params="name parent_link namespace system *origin">
+  <xacro:macro name="imu_generic" params="name parent_link namespace system *origin">
     <link name="${name}_link">
       <inertial>
@@ -14,24 +14,15 @@
     </joint>
     <xacro:if value="${system == 'gz'}">
-      <gazebo reference="${name}_link">
+      <gazebo>
         <plugin filename="gz-sim-imu-system"
           name="gz::sim::systems::Imu">
         </plugin>
-        <sensor name="${name}" type="camera">
-          <camera>
-            <horizontal_fov>1.047</horizontal_fov>
-            <image>
-              <width>1080</width>
-              <height>720</height>
-            </image>
-            <clip>
-              <near>0.1</near>
-              <far>100</far>
-            </clip>
-          </camera>
+      </gazebo>
+      <gazebo reference="${name}_link">
+        <sensor name="${name}" type="imu">
           <always_on>1</always_on>
-          <update_rate>30</update_rate>
+          <update_rate>100</update_rate>
           <visualize>true</visualize>
-          <topic>/${namespace}/${name}/image</topic>
+          <topic>/${namespace}/${name}/imu</topic>
         </sensor>
       </gazebo>

File: foxy_description/urdf/foxy.urdf.xacro (robot description, xacro)
@@ -6,12 +6,21 @@
   <!-- set of properties for internal use (not used by launch) -->
   <xacro:property name="namespace" default="$(arg robot_name)"/>
-  <xacro:property name="root_frame" default="${namespace}/base_link" />
+  <!-- <xacro:property name="root_frame" default="${namespace}/base_link" /> -->
+  <xacro:property name="root_frame" default="base_link" />
   <xacro:property name="ros2_gz_before_renamed" value="${['humble', 'galatic', 'foxy']}"/>
   <xacro:include filename="$(find foxy_description)/urdf/base.xacro"/>
   <xacro:include filename="$(find foxy_description)/sensors/rgb_camera_generic.xacro"/>
+  <xacro:include filename="$(find foxy_description)/sensors/imu_generic.xacro"/>
+  <xacro:include filename="$(find foxy_description)/sensors/lidar_generic.xacro"/>
   <xacro:foxy_base root_frame="${root_frame}"/>
   <xacro:rgb_camera_generic name="front_camera" parent_link="${root_frame}" namespace="${namespace}" system="${xacro.arg('system')}">
     <origin xyz="0.4 0 0.1" rpy="0 0 0" />
   </xacro:rgb_camera_generic>
+  <xacro:imu_generic name="imu_sensor" parent_link="${root_frame}" namespace="${namespace}" system="${xacro.arg('system')}">
+    <origin xyz="0 0 0" rpy="0 0 0" />
+  </xacro:imu_generic>
+  <xacro:lidar_generic name="lidar_sensor" parent_link="${root_frame}" namespace="${namespace}" system="${xacro.arg('system')}">
+    <origin xyz="0.4 0 0.3" rpy="0 0 0" />
+  </xacro:lidar_generic>
   <xacro:if value="${xacro.arg('system') == 'gz' and xacro.arg('distro') in ros2_gz_before_renamed}">
     <!-- the plugin was renamed to gz_ros2_control from Iron -->
