Commit message: rename and rearrange frames

File: foxy_description/urdf/base.xacro (robot description, xacro)
@@ -1,7 +1,10 @@
 <?xml-model href="https://raw.githubusercontent.com/harleylara/urdfdom/refs/heads/movespecification/xsd/urdf.xsd"?>
 <robot name="foxy_base" xmlns:xacro="http://www.ros.org/wiki/xacro">
-  <!-- params description -->
-  <!-- name: prefix the robot root frame -->
-  <xacro:macro name="foxy_base" params="name">
+  <!-- params description for xacro component -->
+  <!-- prefix: prefix the root frame -->
+  <xacro:macro name="foxy_base" params="prefix">
+    <!-- properties -->
+    <!-- root: name of the root frame of the robot -->
+    <xacro:property name="root" default="${prefix}base_link" />
     <material name="grey">
       <color rgba="0.7 0.7 0.7 1" />
@@ -14,5 +17,5 @@
     </material>
     <link name="base_footprint" />
-    <link name="base_link">
+    <link name="${root}">
       <visual>
         <geometry>
@@ -23,13 +26,9 @@
       </visual>
     </link>
-    <link name="lidar">
-      <visual>
-        <geometry>
-          <cylinder radius="0.1" length="0.05" />
-        </geometry>
-        <origin xyz="0 0 0" rpy="0 0 0" />
-        <material name="white" />
-      </visual>
-    </link>
+    <joint name="base_joint" type="fixed">
+      <parent link="${root}" />
+      <child link="base_footprint" />
+      <origin xyz="0 0 -0.1" rpy="0 0 0" />
+    </joint>
     <link name="left_wheel">
       <visual>
@@ -59,26 +58,16 @@
       </visual>
     </link>
-    <joint name="base_joint" type="fixed">
-      <parent link="base_footprint" />
-      <child link="base_link" />
-      <origin xyz="0 0 0.1" rpy="0 0 0" />
-    </joint>
-    <joint name="base_lidar_joint" type="fixed">
-      <parent link="base_link" />
-      <child link="lidar" />
-      <origin xyz="0 0 0.225" rpy="0 0 0" />
-    </joint>
     <joint name="base_left_wheel_joint" type="fixed">
-      <parent link="base_link" />
+      <parent link="${root}" />
       <child link="left_wheel" />
       <origin xyz="-0.15 0.225 0" rpy="0 0 0" />
     </joint>
     <joint name="base_right_wheel_joint" type="fixed">
-      <parent link="base_link" />
+      <parent link="${root}" />
       <child link="right_wheel" />
       <origin xyz="-0.15 -0.225 0" rpy="0 0 0" />
     </joint>
     <joint name="base_caster_wheel_joint" type="fixed">
-      <parent link="base_link" />
+      <parent link="${root}" />
       <child link="caster_wheel" />
       <origin xyz="0.2 0 -0.05" rpy="0 0 0" />

File: foxy_description/urdf/foxy.urdf.xacro (robot description, xacro)
@@ -3,5 +3,8 @@
   <!-- The following set of ARGUMENTS are used by launch -->
   <xacro:arg name="robot_name" default="default"/>
-  <xacro:include filename="$(find foxy_description)/urdf/foxy_base.xacro"/>
-  <xacro:foxy_base/>
+  <!-- set of properties for internal use (not used by launch) -->
+  <xacro:property name="namespace" default="$(arg robot_name)"/>
+  <xacro:property name="prefix" default="${namespace}_" />
+  <xacro:include filename="$(find foxy_description)/urdf/base.xacro"/>
+  <xacro:foxy_base prefix="${prefix}"/>
 </robot>

Commit message: change joints type

File: foxy_description/urdf/base.xacro (robot description, xacro)
@@ -58,13 +58,15 @@
       </visual>
     </link>
-    <joint name="base_left_wheel_joint" type="fixed">
+    <joint name="base_left_wheel_joint" type="continuous">
       <parent link="${root}" />
       <child link="left_wheel" />
       <origin xyz="-0.15 0.225 0" rpy="0 0 0" />
+      <axis xyz="0 1 0"/>
     </joint>
-    <joint name="base_right_wheel_joint" type="fixed">
+    <joint name="base_right_wheel_joint" type="continuous">
       <parent link="${root}" />
       <child link="right_wheel" />
       <origin xyz="-0.15 -0.225 0" rpy="0 0 0" />
+      <axis xyz="0 1 0"/>
     </joint>
     <joint name="base_caster_wheel_joint" type="fixed">

Commit message: change root frame to main file

File: foxy_description/urdf/base.xacro (robot description, xacro)
@@ -2,9 +2,6 @@
 <robot name="foxy_base" xmlns:xacro="http://www.ros.org/wiki/xacro">
   <!-- params description for xacro component -->
-  <!-- prefix: prefix the root frame -->
-  <xacro:macro name="foxy_base" params="prefix">
-    <!-- properties -->
-    <!-- root: name of the root frame of the robot -->
-    <xacro:property name="root" default="${prefix}base_link" />
+  <!-- root_frame: name of the root link frame -->
+  <xacro:macro name="foxy_base" params="root_frame">
     <material name="grey">
       <color rgba="0.7 0.7 0.7 1" />
@@ -17,5 +14,5 @@
     </material>
     <link name="base_footprint" />
-    <link name="${root}">
+    <link name="${root_frame}">
       <visual>
         <geometry>
@@ -27,5 +24,5 @@
     </link>
     <joint name="base_joint" type="fixed">
-      <parent link="${root}" />
+      <parent link="${root_frame}" />
       <child link="base_footprint" />
       <origin xyz="0 0 -0.1" rpy="0 0 0" />
@@ -59,5 +56,5 @@
     </link>
     <joint name="base_left_wheel_joint" type="continuous">
-      <parent link="${root}" />
+      <parent link="${root_frame}" />
       <child link="left_wheel" />
       <origin xyz="-0.15 0.225 0" rpy="0 0 0" />
@@ -65,5 +62,5 @@
     </joint>
     <joint name="base_right_wheel_joint" type="continuous">
-      <parent link="${root}" />
+      <parent link="${root_frame}" />
       <child link="right_wheel" />
       <origin xyz="-0.15 -0.225 0" rpy="0 0 0" />
@@ -71,5 +68,5 @@
     </joint>
     <joint name="base_caster_wheel_joint" type="fixed">
-      <parent link="${root}" />
+      <parent link="${root_frame}" />
       <child link="caster_wheel" />
       <origin xyz="0.2 0 -0.05" rpy="0 0 0" />

File: foxy_description/urdf/foxy.urdf.xacro (robot description, xacro)
@@ -5,6 +5,6 @@
   <!-- set of properties for internal use (not used by launch) -->
   <xacro:property name="namespace" default="$(arg robot_name)"/>
-  <xacro:property name="prefix" default="${namespace}_" />
+  <xacro:property name="root_frame" default="${namespace}_base_link" />
   <xacro:include filename="$(find foxy_description)/urdf/base.xacro"/>
-  <xacro:foxy_base prefix="${prefix}"/>
+  <xacro:foxy_base root_frame="${root_frame}"/>
 </robot>

Commit message: add gz_control_plugin

File: foxy_description/urdf/base.xacro (robot description, xacro)
@@ -1,3 +1,2 @@
-<?xml-model href="https://raw.githubusercontent.com/harleylara/urdfdom/refs/heads/movespecification/xsd/urdf.xsd"?>
 <robot name="foxy_base" xmlns:xacro="http://www.ros.org/wiki/xacro">
   <!-- params description for xacro component -->
@@ -22,4 +21,9 @@
         <material name="green" />
       </visual>
+      <collision>
+        <geometry>
+          <box size="0.6 0.4 0.2" />
+        </geometry>
+      </collision>
     </link>
     <joint name="base_joint" type="fixed">
@@ -36,4 +40,13 @@
         <material name="grey" />
       </visual>
+      <collision>
+        <geometry>
+          <cylinder radius="0.1" length="0.05" />
+        </geometry>
+      </collision>
+      <inertial>
+        <mass value="1"/>
+        <inertia ixx="0.4" ixy="0.0" ixz="0.0" iyy="0.4" iyz="0.0" izz="0.2"/>
+      </inertial>
     </link>
     <link name="right_wheel">
@@ -45,4 +58,13 @@
         <material name="grey" />
       </visual>
+      <collision>
+        <geometry>
+          <cylinder radius="0.1" length="0.05" />
+        </geometry>
+      </collision>
+      <inertial>
+        <mass value="1"/>
+        <inertia ixx="0.4" ixy="0.0" ixz="0.0" iyy="0.4" iyz="0.0" izz="0.2"/>
+      </inertial>
     </link>
     <link name="caster_wheel">
@@ -54,4 +76,13 @@
         <material name="grey" />
       </visual>
+      <collision>
+        <geometry>
+          <sphere radius="0.05" />
+        </geometry>
+      </collision>
+      <inertial>
+        <mass value="0.01"/>
+        <inertia ixx="0.4" ixy="0.0" ixz="0.0" iyy="0.4" iyz="0.0" izz="0.2"/>
+      </inertial>
     </link>
     <joint name="base_left_wheel_joint" type="continuous">

File: foxy_description/urdf/foxy.urdf.xacro (robot description, xacro)
@@ -1,3 +1,2 @@
-<?xml-model href="https://raw.githubusercontent.com/harleylara/urdfdom/refs/heads/movespecification/xsd/urdf.xsd"?>
 <robot name="robot" xmlns:xacro="http://www.ros.org/wiki/xacro">
   <!-- The following set of ARGUMENTS are used by launch -->
@@ -12,5 +11,5 @@
     <ros2_control name="GazeboSimSystem" type="system">
       <hardware>
-        <plugin>gz_ros2_control/GazeboSimSystem</plugin>
+        <plugin>ign_ros2_control/IgnitionSystem</plugin>
       </hardware>
       <joint name="base_left_wheel_joint">
@@ -32,7 +31,8 @@
     </ros2_control>
     <gazebo>
-      <plugin filename="gz_ros2_control-system" name="gz_ros2_control::GazeboSimROS2ControlPlugin">
+      <!-- the plugin was renamed to gz_ros2_control from Iron -->
+      <plugin filename="ign_ros2_control-system" name="ign_ros2_control::IgnitionROS2ControlPlugin">
         <ros>
-          <namespace>"${namespace}"</namespace>
+          <namespace>${namespace}</namespace>
         </ros>
         <parameters>$(find foxy_bringup)/config/controllers.yaml</parameters>

Commit message: add working demo diff drive

File: foxy_description/urdf/base.xacro (robot description, xacro)
@@ -15,11 +15,12 @@
     <link name="${root_frame}">
       <visual>
+        <origin xyz="0 0 0.1" rpy="0 0 0" />
         <geometry>
           <box size="0.6 0.4 0.2" />
         </geometry>
-        <origin xyz="0 0 0.1" rpy="0 0 0" />
         <material name="green" />
       </visual>
       <collision>
+        <origin xyz="0 0 0.1" rpy="0 0 0" />
         <geometry>
           <box size="0.6 0.4 0.2" />
@@ -34,11 +35,12 @@
     <link name="left_wheel">
       <visual>
+        <origin xyz="0 0 0" rpy="1.57 0 0" />
         <geometry>
           <cylinder radius="0.1" length="0.05" />
         </geometry>
-        <origin xyz="0 0 0" rpy="1.57 0 0" />
         <material name="grey" />
       </visual>
       <collision>
+        <origin xyz="0 0 0" rpy="1.57 0 0" />
         <geometry>
           <cylinder radius="0.1" length="0.05" />
@@ -46,4 +48,5 @@
       </collision>
       <inertial>
+        <origin xyz="0 0 0" rpy="1.57 0 0" />
         <mass value="1"/>
         <inertia ixx="0.4" ixy="0.0" ixz="0.0" iyy="0.4" iyz="0.0" izz="0.2"/>
@@ -52,11 +55,12 @@
     <link name="right_wheel">
       <visual>
+        <origin xyz="0 0 0" rpy="1.57 0 0" />
         <geometry>
           <cylinder radius="0.1" length="0.05" />
         </geometry>
-        <origin xyz="0 0 0" rpy="1.57 0 0" />
         <material name="grey" />
       </visual>
       <collision>
+        <origin xyz="0 0 0" rpy="1.57 0 0" />
         <geometry>
           <cylinder radius="0.1" length="0.05" />
@@ -64,4 +68,5 @@
       </collision>
       <inertial>
+        <origin xyz="0 0 0" rpy="1.57 0 0" />
         <mass value="1"/>
         <inertia ixx="0.4" ixy="0.0" ixz="0.0" iyy="0.4" iyz="0.0" izz="0.2"/>
@@ -86,15 +91,17 @@
       </inertial>
     </link>
-    <joint name="base_left_wheel_joint" type="continuous">
+    <joint name="left_wheel_joint" type="continuous">
       <parent link="${root_frame}" />
       <child link="left_wheel" />
-      <origin xyz="-0.15 0.225 0" rpy="0 0 0" />
+      <origin xyz="-0.15 0.25 0" rpy="0 0 0" />
       <axis xyz="0 1 0"/>
+      <dynamics damping="0.2"/>
     </joint>
-    <joint name="base_right_wheel_joint" type="continuous">
+    <joint name="right_wheel_joint" type="continuous">
       <parent link="${root_frame}" />
       <child link="right_wheel" />
-      <origin xyz="-0.15 -0.225 0" rpy="0 0 0" />
+      <origin xyz="-0.15 -0.25 0" rpy="0 0 0" />
       <axis xyz="0 1 0"/>
+      <dynamics damping="0.2"/>
     </joint>
     <joint name="base_caster_wheel_joint" type="fixed">

File: foxy_description/urdf/foxy.urdf.xacro (robot description, xacro)
@@ -6,5 +6,5 @@
   <!-- set of properties for internal use (not used by launch) -->
   <xacro:property name="namespace" default="$(arg robot_name)"/>
-  <xacro:property name="root_frame" default="${namespace}_base_link" />
+  <xacro:property name="root_frame" default="${namespace}/base_link" />
   <xacro:property name="ros2_gz_before_renamed" value="${['humble', 'galatic', 'foxy']}"/>
   <xacro:include filename="$(find foxy_description)/urdf/base.xacro"/>
@@ -16,5 +16,5 @@
         <plugin>ign_ros2_control/IgnitionSystem</plugin>
       </hardware>
-      <joint name="base_left_wheel_joint">
+      <joint name="left_wheel_joint">
         <command_interface name="velocity">
           <param name="min">-1</param>
@@ -24,5 +24,5 @@
         <state_interface name="velocity"/>
       </joint>
-      <joint name="base_right_wheel_joint">
+      <joint name="right_wheel_joint">
         <command_interface name="velocity">
           <param name="min">-1</param>

Commit message: add mass to base

File: foxy_description/urdf/base.xacro (robot description, xacro)
@@ -27,4 +27,9 @@
         </geometry>
       </collision>
+      <inertial>
+        <origin xyz="0 0 0" rpy="0 0 0" />
+        <mass value="1"/>
+        <inertia ixx="0.4" ixy="0.0" ixz="0.0" iyy="0.4" iyz="0.0" izz="0.2"/>
+      </inertial>
     </link>
     <joint name="base_joint" type="fixed">

Commit message: fix wheel position

File: foxy_description/urdf/base.xacro (robot description, xacro)
@@ -99,5 +99,5 @@
       <parent link="${root_frame}" />
       <child link="left_wheel" />
-      <origin xyz="-0.15 0.25 0" rpy="0 0 0" />
+      <origin xyz="0.15 0.25 0" rpy="0 0 0" />
       <axis xyz="0 1 0"/>
       <dynamics damping="0.2"/>
@@ -106,5 +106,5 @@
       <parent link="${root_frame}" />
       <child link="right_wheel" />
-      <origin xyz="-0.15 -0.25 0" rpy="0 0 0" />
+      <origin xyz="0.15 -0.25 0" rpy="0 0 0" />
       <axis xyz="0 1 0"/>
       <dynamics damping="0.2"/>
@@ -113,5 +113,5 @@
       <parent link="${root_frame}" />
       <child link="caster_wheel" />
-      <origin xyz="0.2 0 -0.05" rpy="0 0 0" />
+      <origin xyz="-0.2 0 -0.05" rpy="0 0 0" />
     </joint>
   </xacro:macro>

Commit message: refactor robot size and mass

File: foxy_description/urdf/base.xacro (robot description, xacro)
@@ -1,3 +1,41 @@
 <robot name="foxy_base" xmlns:xacro="http://www.ros.org/wiki/xacro">
+  <xacro:property name="base_width" value="0.07"/>
+  <xacro:property name="base_length" value="0.13"/>
+  <xacro:property name="base_height" value="0.08"/>
+  <xacro:property name="wheel_radius" value="0.033"/>
+  <xacro:property name="wheel_width" value="0.025"/>
+  <xacro:property name="wheel_separation" value="0.101"/>
+  <xacro:property name="wheel_zoff" value="0.05"/>
+  <xacro:property name="wheel_xoff" value="0.04"/>
+  <xacro:property name="caster_radius" value="0.009"/>
+  <xacro:property name="caster_zoff" value="0.032"/>
+  <xacro:property name="caster_xoff" value="-0.043"/>
+  <xacro:include filename="$(find foxy_description)/urdf/utils.xacro"/>
+  <xacro:macro name="wheel" params="prefix parent x_reflect y_reflect">
+    <link name="${prefix}_link">
+      <visual>
+        <origin xyz="0 0 0" rpy="${pi/2} 0 0"/>
+        <geometry>
+          <cylinder radius="${wheel_radius}" length="${wheel_width}"/>
+        </geometry>
+        <material name="Gray">
+          <color rgba="0.5 0.5 0.5 1.0"/>
+        </material>
+      </visual>
+      <collision>
+        <origin xyz="0 0 0" rpy="${pi/2} 0 0"/>
+        <geometry>
+          <cylinder radius="${wheel_radius}" length="${wheel_width}"/>
+        </geometry>
+      </collision>
+      <xacro:cylinder_inertia m="0.05" r="${wheel_radius}" h="${wheel_width}"/>
+    </link>
+    <joint name="${prefix}_joint" type="continuous">
+      <parent link="${parent}"/>
+      <child link="${prefix}_link"/>
+      <origin xyz="${x_reflect*wheel_xoff} ${y_reflect*(wheel_separation/2)} ${-wheel_zoff}" rpy="0 0 0"/>
+      <axis xyz="0 1 0"/>
+    </joint>
+  </xacro:macro>
   <!-- params description for xacro component -->
   <!-- root_frame: name of the root link frame -->
@@ -12,8 +50,12 @@
       <color rgba="1 1 1 1" />
     </material>
-    <link name="base_footprint" />
+    <link name="base_footprint">
+      <xacro:box_inertia m="0.5" w="${base_width}" d="${base_length}" h="${base_height}"/>
+    </link>
     <link name="${root_frame}">
       <visual>
-        <origin xyz="0 0 0.1" rpy="0 0 0" />
+        <geometry>
+          <box size="${base_length} ${base_width} ${base_height}"/>
+        </geometry>
         <geometry>
           <box size="0.6 0.4 0.2" />
@@ -22,96 +64,34 @@
       </visual>
       <collision>
-        <origin xyz="0 0 0.1" rpy="0 0 0" />
         <geometry>
-          <box size="0.6 0.4 0.2" />
+          <box size="${base_length} ${base_width} ${base_height}"/>
         </geometry>
       </collision>
-      <inertial>
-        <origin xyz="0 0 0" rpy="0 0 0" />
-        <mass value="1"/>
-        <inertia ixx="0.4" ixy="0.0" ixz="0.0" iyy="0.4" iyz="0.0" izz="0.2"/>
-      </inertial>
     </link>
     <joint name="base_joint" type="fixed">
       <parent link="${root_frame}" />
       <child link="base_footprint" />
-      <origin xyz="0 0 -0.1" rpy="0 0 0" />
+      <origin xyz="0 0 ${-(wheel_radius+wheel_zoff)}" rpy="0 0 0" />
     </joint>
-    <link name="left_wheel">
+    <xacro:wheel prefix="left_wheel" parent="${root_frame}" x_reflect="1" y_reflect="1" />
+    <xacro:wheel prefix="right_wheel" parent="${root_frame}" x_reflect="1" y_reflect="-1" />
+    <link name="caster_wheel">
       <visual>
-        <origin xyz="0 0 0" rpy="1.57 0 0" />
         <geometry>
-          <cylinder radius="0.1" length="0.05" />
+          <sphere radius="${caster_radius}" />
         </geometry>
         <material name="grey" />
       </visual>
       <collision>
-        <origin xyz="0 0 0" rpy="1.57 0 0" />
         <geometry>
-          <cylinder radius="0.1" length="0.05" />
+          <sphere radius="${caster_radius}" />
         </geometry>
       </collision>
-      <inertial>
-        <origin xyz="0 0 0" rpy="1.57 0 0" />
-        <mass value="1"/>
-        <inertia ixx="0.4" ixy="0.0" ixz="0.0" iyy="0.4" iyz="0.0" izz="0.2"/>
-      </inertial>
+      <xacro:sphere_inertia m="0.01" r="${caster_radius}"/>
     </link>
-    <link name="right_wheel">
-      <visual>
-        <origin xyz="0 0 0" rpy="1.57 0 0" />
-        <geometry>
-          <cylinder radius="0.1" length="0.05" />
-        </geometry>
-        <material name="grey" />
-      </visual>
-      <collision>
-        <origin xyz="0 0 0" rpy="1.57 0 0" />
-        <geometry>
-          <cylinder radius="0.1" length="0.05" />
-        </geometry>
-      </collision>
-      <inertial>
-        <origin xyz="0 0 0" rpy="1.57 0 0" />
-        <mass value="1"/>
-        <inertia ixx="0.4" ixy="0.0" ixz="0.0" iyy="0.4" iyz="0.0" izz="0.2"/>
-      </inertial>
-    </link>
-    <link name="caster_wheel">
-      <visual>
-        <geometry>
-          <sphere radius="0.05" />
-        </geometry>
-        <origin xyz="0 0 0" rpy="0 0 0" />
-        <material name="grey" />
-      </visual>
-      <collision>
-        <geometry>
-          <sphere radius="0.05" />
-        </geometry>
-      </collision>
-      <inertial>
-        <mass value="0.01"/>
-        <inertia ixx="0.4" ixy="0.0" ixz="0.0" iyy="0.4" iyz="0.0" izz="0.2"/>
-      </inertial>
-    </link>
-    <joint name="left_wheel_joint" type="continuous">
-      <parent link="${root_frame}" />
-      <child link="left_wheel" />
-      <origin xyz="0.15 0.25 0" rpy="0 0 0" />
-      <axis xyz="0 1 0"/>
-      <dynamics damping="0.2"/>
-    </joint>
-    <joint name="right_wheel_joint" type="continuous">
-      <parent link="${root_frame}" />
-      <child link="right_wheel" />
-      <origin xyz="0.15 -0.25 0" rpy="0 0 0" />
-      <axis xyz="0 1 0"/>
-      <dynamics damping="0.2"/>
-    </joint>
     <joint name="base_caster_wheel_joint" type="fixed">
       <parent link="${root_frame}" />
       <child link="caster_wheel" />
-      <origin xyz="-0.2 0 -0.05" rpy="0 0 0" />
+      <origin xyz="${caster_xoff} 0 -${(wheel_radius+wheel_zoff)-caster_radius}" rpy="0 0 0" />
     </joint>
   </xacro:macro>

File: foxy_description/urdf/foxy.urdf.xacro (robot description, xacro)
@@ -15,5 +15,5 @@
   <xacro:foxy_base root_frame="${root_frame}"/>
   <xacro:rgb_camera_generic name="front_camera" parent_link="${root_frame}" namespace="${namespace}" system="${xacro.arg('system')}">
-    <origin xyz="0.4 0 0.1" rpy="0 0 0" />
+    <origin xyz="0.075 0 0.07" rpy="0 0 0" />
   </xacro:rgb_camera_generic>
   <xacro:imu_generic name="imu_sensor" parent_link="${root_frame}" namespace="${namespace}" system="${xacro.arg('system')}">
@@ -21,5 +21,5 @@
   </xacro:imu_generic>
   <xacro:lidar_generic name="lidar_sensor" parent_link="${root_frame}" namespace="${namespace}" system="${xacro.arg('system')}">
-    <origin xyz="0.4 0 0.3" rpy="0 0 0" />
+    <origin xyz="0 0 0.12" rpy="0 0 0" />
   </xacro:lidar_generic>
   <xacro:if value="${xacro.arg('system') == 'gz' and xacro.arg('distro') in ros2_gz_before_renamed}">
