Commit message: add conditional for system

File: foxy_description/urdf/foxy.urdf.xacro (robot description, xacro)
@@ -3,4 +3,5 @@
   <!-- The following set of ARGUMENTS are used by launch -->
   <xacro:arg name="robot_name" default="default"/>
+  <xacro:arg name="system" default="none"/>
   <!-- set of properties for internal use (not used by launch) -->
   <xacro:property name="namespace" default="$(arg robot_name)"/>
@@ -8,3 +9,34 @@
   <xacro:include filename="$(find foxy_description)/urdf/base.xacro"/>
   <xacro:foxy_base root_frame="${root_frame}"/>
+  <xacro:if value="${xacro.arg('system') == 'gz'}">
+    <ros2_control name="GazeboSimSystem" type="system">
+      <hardware>
+        <plugin>gz_ros2_control/GazeboSimSystem</plugin>
+      </hardware>
+      <joint name="base_left_wheel_joint">
+        <command_interface name="velocity">
+          <param name="min">-1</param>
+          <param name="max">1</param>
+        </command_interface>
+        <state_interface name="position"/>
+        <state_interface name="velocity"/>
+      </joint>
+      <joint name="base_right_wheel_joint">
+        <command_interface name="velocity">
+          <param name="min">-1</param>
+          <param name="max">1</param>
+        </command_interface>
+        <state_interface name="position"/>
+        <state_interface name="velocity"/>
+      </joint>
+    </ros2_control>
+    <gazebo>
+      <plugin filename="gz_ros2_control-system" name="gz_ros2_control::GazeboSimROS2ControlPlugin">
+        <ros>
+          <namespace>"${namespace}"</namespace>
+        </ros>
+        <parameters>$(find foxy_bringup)/config/controllers.yaml</parameters>
+      </plugin>
+    </gazebo>
+  </xacro:if>
 </robot>

Commit message: working example of bringup

File: foxy_description/urdf/foxy.urdf.xacro (robot description, xacro)
@@ -3,10 +3,13 @@
   <xacro:arg name="robot_name" default="default"/>
   <xacro:arg name="system" default="none"/>
+  <xacro:arg name="distro" default="none"/> <!-- for internal use -->
   <!-- set of properties for internal use (not used by launch) -->
   <xacro:property name="namespace" default="$(arg robot_name)"/>
   <xacro:property name="root_frame" default="${namespace}_base_link" />
+  <xacro:property name="ros2_gz_before_renamed" value="${['humble', 'galatic', 'foxy']}"/>
   <xacro:include filename="$(find foxy_description)/urdf/base.xacro"/>
   <xacro:foxy_base root_frame="${root_frame}"/>
-  <xacro:if value="${xacro.arg('system') == 'gz'}">
+  <xacro:if value="${xacro.arg('system') == 'gz' and xacro.arg('distro') in ros2_gz_before_renamed}">
+    <!-- the plugin was renamed to gz_ros2_control from Iron -->
     <ros2_control name="GazeboSimSystem" type="system">
       <hardware>
@@ -31,5 +34,4 @@
     </ros2_control>
     <gazebo>
-      <!-- the plugin was renamed to gz_ros2_control from Iron -->
       <plugin filename="ign_ros2_control-system" name="ign_ros2_control::IgnitionROS2ControlPlugin">
         <ros>

Commit message: add rgb camera suppport for gz

File: foxy_description/urdf/foxy.urdf.xacro (robot description, xacro)
@@ -9,5 +9,9 @@
   <xacro:property name="ros2_gz_before_renamed" value="${['humble', 'galatic', 'foxy']}"/>
   <xacro:include filename="$(find foxy_description)/urdf/base.xacro"/>
+ :<xacro:include filename="$(find foxy_description)/sensors/rgb_camera_generic.xacro"/>
   <xacro:foxy_base root_frame="${root_frame}"/>
+  <xacro:rgb_camera_generic name="front_camera" parent_link="${root_frame}" namespace="${namespace}" system="${xacro.arg('system')}">
+    <origin xyz="0.4 0 0.1" rpy="0 0 0" />
+  </xacro:rgb_camera_generic>
   <xacro:if value="${xacro.arg('system') == 'gz' and xacro.arg('distro') in ros2_gz_before_renamed}">
     <!-- the plugin was renamed to gz_ros2_control from Iron -->
@@ -34,4 +38,8 @@
     </ros2_control>
     <gazebo>
+      <!-- inserted at the top level of the <model> tag -->
+      <plugin filename="ignition-gazebo-sensors-system" name="ignition::gazebo::systems::Sensors">
+        <render_engine>ogre</render_engine>
+      </plugin>
       <plugin filename="ign_ros2_control-system" name="ign_ros2_control::IgnitionROS2ControlPlugin">
         <ros>

Commit message: add camera pitch

File: foxy_description/urdf/foxy.urdf.xacro (robot description, xacro)
@@ -15,5 +15,5 @@
   <xacro:foxy_base root_frame="${root_frame}"/>
   <xacro:rgb_camera_generic name="front_camera" parent_link="${root_frame}" namespace="${namespace}" system="${xacro.arg('system')}">
-    <origin xyz="0.075 0 0.07" rpy="0 0 0" />
+    <origin xyz="0.075 0 0.07" rpy="0.0 0.13 0" />
   </xacro:rgb_camera_generic>
   <xacro:imu_generic name="imu_sensor" parent_link="${root_frame}" namespace="${namespace}" system="${xacro.arg('system')}">
